Commit message: implemented tracks using Gazebo's TrackedVehicle plugin

File: jo_description/urdf/front_depth.xacro (robot description, xacro)
@@ -7,36 +7,37 @@
     <xacro:property name="b2c_R" value="0.0" />
     <xacro:property name="b2c_P" value="0.0" />
-    <xacro:property name="b2c_Y" value="${PI}" />
+    <xacro:property name="b2c_Y" value="0.0" />
     <xacro:property name="camera_mass" value="0.125" />
-    <xacro:property name="camera_len_rad" value="0.0508" />
-    <xacro:property name="camera_len_h" value="0.055" />
+    <xacro:property name="camera_height" value="0.03" />
+    <xacro:property name="camera_len" value="0.14" />
+    <xacro:property name="camera_depth" value="0.03" />
     <xacro:include filename="$(find jo_description)/urdf/inertial_macros.xacro" />
-    <xacro:macro name="d455" params="namespace">
-        <joint name="base2camera" type="fixed">
+    <xacro:macro name="front_depth" params="namespace">
+        <joint name="base2front_camera" type="fixed">
             <parent link="base_link"/>
-            <child link="camera_link"/>
-            <origin xyz="${b2c_x} ${b2c_y} ${b2c_z}" rpy="${b2c_R} ${b2c_P} ${b2c_Y}"/>
+            <child link="front_camera_link"/>
+            <origin xyz="${-b2c_x + 0.03} ${b2c_y} ${b2c_z}" rpy="${b2c_R} ${b2c_P} ${b2c_Y}"/>
         </joint>
-        <link name="camera_link">
-            <collision>
-                <origin xyz="0 0 0" rpy="0 0 0"/>
-                <geometry>
-                    <cylinder radius="${camera_len_rad}" length="${camera_len_h}"/>
-                </geometry>
-            </collision>
+        <link name="front_camera_link">
             <visual>
                 <origin xyz="0 0 0" rpy="0 ${PI/2} 0"/>
                 <geometry>
-                    <cylinder radius="${camera_len_rad}" length="${camera_len_h}"/>
+                    <box size="${camera_depth} ${camera_len} ${camera_height}"/>
                 </geometry>
-                <material name="orange"/>
+                <material name="gray"/>
             </visual>
-            <xacro:inertial_cylinder mass="${camera_mass}" radius="${camera_len_rad}" length="${camera_len_h}">
-                    <origin xyz="0 0 0" rpy="0 0 0"/>
-            </xacro:inertial_cylinder>
+            <collision>
+                <origin xyz="0 0 0" rpy="0 ${PI/2} 0"/>
+                <geometry>
+                    <box size="${camera_depth} ${camera_len} ${camera_height}"/>
+                </geometry>
+            </collision>
+            <xacro:inertial_box mass="${camera_mass}" x="${camera_depth}" y="${camera_len}" z="${camera_height}">
+                    <origin xyz="0 0 0" rpy="0 ${PI/2} 0"/>
+            </xacro:inertial_box>
         </link>
-        <gazebo reference="camera_link">
-            <sensor name="d455" type="rgbd_camera">
-                <gz_frame_id>camera_link</gz_frame_id>
+        <gazebo reference="front_camera_link">
+            <sensor name="front_d455" type="rgbd_camera">
+                <gz_frame_id>front_camera_link</gz_frame_id>
                 <always_on>true</always_on>
                 <update_rate>30</update_rate>
@@ -62,8 +63,8 @@
                 </clip>
                 </depth_camera>
-                <topic>camera</topic>
+                <topic>front_camera</topic>
             </sensor>
             </gazebo>
     </xacro:macro>
-    <xacro:d455 namespace=""/>
+    <xacro:front_depth namespace=""/>
 </robot>

File: jo_description/urdf/imu.xacro (robot description, xacro)
@@ -9,7 +9,7 @@
     <xacro:property name="b2i_Y" value="0.0" />
     <xacro:property name="imu_mass" value="0.01" />
-    <xacro:property name="imu_len_x" value="0.01" />
-    <xacro:property name="imu_len_y" value="0.01" />
-    <xacro:property name="imu_len_z" value="0.01" />
+    <xacro:property name="imu_len_x" value="0.05" />
+    <xacro:property name="imu_len_y" value="0.05" />
+    <xacro:property name="imu_len_z" value="0.05" />
     <xacro:include filename="$(find jo_description)/urdf/inertial_macros.xacro" />
     <xacro:macro name="imu_sensor" params="">

File: jo_description/urdf/jo_main.urdf.xacro (robot description, xacro)
@@ -1,19 +1,61 @@
 <?xml version="1.0"?>
 <robot xmlns:xacro="http://www.ros.org/wiki/xacro"  name="jo">
-    <xacro:arg name="use_ros2_control" default="true"/>
-    <xacro:arg name="use_sim_time" default="false"/>
     <xacro:include filename="robot_core.xacro" />
-    <xacro:include filename="ros2_control.xacro" />
+    <xacro:include filename="track.xacro" />
+    <xacro:track side="left"/>
+    <xacro:track side="right"/>
+    <!-- <xacro:include filename="ros2_control.xacro" /> -->
     <xacro:include filename="velodyne.xacro" />
-    <xacro:include filename="D455.xacro" />
+    <xacro:include filename="front_depth.xacro" />
+    <xacro:include filename="back_depth.xacro" />
     <xacro:include filename="imu.xacro" />
-    <!-- <xacro:if value="$(arg use_ros2_control)">
-        <xacro:include filename="ros2_control.xacro" />
-    </xacro:if>
-    <xacro:unless value="$(arg use_ros2_control)">
-        <xacro:include filename="gazebo_control.xacro" />
-    </xacro:unless>
-    <xacro:include filename="lidar.xacro" />
-    <xacro:include filename="camera.xacro" />
-    <xacro:include filename="depth_camera.xacro" /> -->
+    <!-- TrackedVehicle instantiation; the track links need to be instantiated separately -->
+    <gazebo>
+        <plugin filename="gz-sim-tracked-vehicle-system"
+                name="gz::sim::systems::TrackedVehicle">
+            <!-- Left track links -->
+            <left_track>
+                <link>left_bottom_belt</link>
+            </left_track>
+            <left_track>
+                <link>front_left_roller</link>
+            </left_track>
+            <left_track>
+                <link>back_left_roller</link>
+            </left_track>
+            <left_track>
+                <link>left_front_bottom_belt</link>
+            </left_track>
+            <!-- Right track links -->
+            <right_track>
+                <link>right_bottom_belt</link>
+            </right_track>
+            <right_track>
+                <link>back_right_roller</link>
+            </right_track>
+            <right_track>
+                <link>front_right_roller</link>
+            </right_track>
+            <right_track>
+                <link>right_front_bottom_belt</link>
+            </right_track>
+            <!-- ODOMETRY SEEMS TO NOT WORK FINE -->
+            <!-- Distance between track centerlines -->
+            <tracks_separation>${chassis_width}</tracks_separation>
+            <!-- Used for odometry moment-arm calculation -->
+            <track_height>${back_roller_radius*2}</track_height>
+            <steering_efficiency>0.5</steering_efficiency>
+            <linear_velocity>
+                <max_velocity>2.0</max_velocity>
+                <max_acceleration>5.0</max_acceleration>
+            </linear_velocity>
+            <angular_velocity>
+                <max_velocity>1.5</max_velocity>
+                <max_acceleration>2.5</max_acceleration>
+            </angular_velocity>
+            <frame_id>odom</frame_id>
+            <child_frame_id>base_link</child_frame_id>
+            <odom_publish_frequency>50</odom_publish_frequency>
+        </plugin>
+    </gazebo>
 </robot>

File: jo_description/urdf/robot_core.xacro (robot description, xacro)
@@ -1,58 +1,48 @@
 <?xml version="1.0"?>
-<robot xmlns:xacro="http://www.ros.org/wiki/xacro" >
+<robot xmlns:xacro="http://www.ros.org/wiki/xacro">
     <xacro:include filename="inertial_macros.xacro"/>
-    <xacro:property name="chassis_length" value="1.064"/>
-    <xacro:property name="chassis_width" value="0.545"/>
+    <xacro:property name="chassis_length" value="0.94"/>
+    <xacro:property name="chassis_width" value="0.39"/>
     <xacro:property name="chassis_height" value="0.273"/>
     <xacro:property name="chassis_mass" value="140.0"/>
-    <xacro:property name="wheel_radius" value="0.1"/>
-    <xacro:property name="wheel_thickness" value="0.15"/>
-    <xacro:property name="wheel_mass" value="20.0"/>
-    <xacro:property name="wheel_offset_x" value="0.532"/>
-    <xacro:property name="wheel_offset_y" value="${chassis_width/2 + wheel_thickness/2}"/>
-    <xacro:property name="wheel_offset_z" value="${chassis_height}"/>
-    <xacro:property name="wheel_spacing" value="0.4"/>
-    <xacro:property name="caster_wheel_radius" value="${wheel_radius}"/>
-    <xacro:property name="caster_wheel_mass" value="0.01"/>
-    <xacro:property name="caster_wheel_offset_x" value="${chassis_length/2 - caster_wheel_radius}"/>
-    <xacro:property name="caster_wheel_offset_z" value="${chassis_height}"/>
-    <material name="white">
-        <color rgba="1 1 1 1" />
-    </material>
-    <material name="orange">
-        <color rgba="1 0.3 0.1 1"/>
-    </material>
-    <material name="blue">
-        <color rgba="0.2 0.2 1 1"/>
-    </material>
-    <material name="black">
-        <color rgba="0 0 0 1"/>
-    </material>
-    <material name="black_t">
-        <color rgba="0 0 0 0.5"/>
-    </material>
-    <material name="red">
-        <color rgba="1 0 0 1"/>
-    </material>
-    <!-- BASE LINK -->
-    <link name="base_link">
-    </link>
-    <!-- BASE_FOOTPRINT LINK -->
+    <xacro:property name="front_chassis2rack" value="0.15"/>
+    <xacro:property name="rack_length" value="0.6"/>
+    <xacro:property name="rack_width" value="0.37"/>
+    <xacro:property name="rack_height" value="0.45"/>
+    <xacro:property name="rack_mass" value="0.0"/>
+    <!-- Lateral offset: center of track from robot centerline -->
+    <xacro:property name="track_offset_y" value="${chassis_width/2 + track_width/2}"/>
+    <!-- Z: bottom of chassis minus half track height = track center sits at ground level -->
+    <xacro:property name="track_offset_z" value="${-chassis_height/2 - track_height/2}"/>
+    <!-- Rack -->
+    <xacro:property name="rack_mass" value="0.1"/>
+    <material name="white">  <color rgba="1 1 1 1"/>         </material>
+    <material name="orange"> <color rgba="1 0.3 0.1 1"/>     </material>
+    <material name="blue">   <color rgba="0.2 0.2 1 1"/>     </material>
+    <material name="black">  <color rgba="0 0 0 1"/>         </material>
+    <material name="black_t"><color rgba="0 0 0 0.9"/>       </material>
+    <material name="red">    <color rgba="1 0 0 1"/>         </material>
+    <material name="gray">    <color rgba="0.5 0.5 0.5 1"/>         </material>
+    <!-- ═══════════════════════════════════════════
+         BASE LINK
+    ═══════════════════════════════════════════ -->
+    <link name="base_link"/>
     <joint name="base_footprint_joint" type="fixed">
         <parent link="base_link"/>
         <child link="base_footprint"/>
-        <origin xyz="0 0 ${-chassis_height - wheel_radius}" rpy="0 0 0"/>
+        <origin xyz="0 0 ${-chassis_height - 0.1}" rpy="0 0 0"/>
     </joint>
-    <link name="base_footprint">
-    </link>
-    <!-- CHASSIS LINK -->
+    <link name="base_footprint"/>
+    <!-- ═══════════════════════════════════════════
+         CHASSIS
+    ═══════════════════════════════════════════ -->
     <joint name="chassis_joint" type="fixed">
         <parent link="base_link"/>
         <child link="chassis"/>
-        <origin xyz="${-wheel_offset_x} 0 ${-chassis_height/2}"/>
+        <origin xyz="${-chassis_length/2} 0 0"/>
     </joint>
     <link name="chassis">
         <visual>
-            <origin xyz="${chassis_length/2} 0 0"/>
+            <origin xyz="${chassis_length/2} 0 ${-chassis_height/2}"/>
             <geometry>
                 <box size="${chassis_length} ${chassis_width} ${chassis_height}"/>
@@ -61,11 +51,12 @@
         </visual>
         <collision>
-            <origin xyz="${chassis_length/2} 0 0"/>
+            <origin xyz="${chassis_length/2} 0 ${-chassis_height/2}"/>
             <geometry>
                 <box size="${chassis_length} ${chassis_width} ${chassis_height}"/>
             </geometry>
         </collision>
-        <xacro:inertial_box mass="${chassis_mass}" x="${chassis_length}" y="${chassis_width}" z="${chassis_height}">
-            <origin xyz="${chassis_length/2} 0 0" rpy="0 0 0"/>
+        <xacro:inertial_box mass="${chassis_mass}"
+                            x="${chassis_length}" y="${chassis_width}" z="${chassis_height}">
+            <origin xyz="${chassis_length/2} 0 ${-chassis_height/2}" rpy="0 0 0"/>
         </xacro:inertial_box>
     </link>
@@ -73,161 +64,17 @@
         <material>Gazebo/White</material>
     </gazebo>
-    <!-- LEFT WHEEL LINK -->
-    <joint name="left_wheel_center_joint" type="continuous">
+    <!-- ═══════════════════════════════════════════
+         RACK
+    ═══════════════════════════════════════════ -->
+    <joint name="base2rack" type="fixed">
         <parent link="base_link"/>
-        <child link="left_wheel_center"/>
-        <origin xyz="0 ${wheel_offset_y} ${-wheel_offset_z}" rpy="-${pi/2} 0 0" />
-        <axis xyz="0 0 1"/>
+        <child link="rack"/>
+        <origin xyz="${-rack_length/2 - front_chassis2rack + chassis_length/2} 0 ${rack_height/2 + 0.02}"/>
     </joint>
-    <link name="left_wheel_center">
-        <visual>
-            <geometry>
-                <cylinder radius="${wheel_radius}" length="${wheel_thickness}"/>
-            </geometry>
-            <material name="black"/>
-        </visual>
-        <collision>
-            <geometry>
-                <sphere radius="${wheel_radius}"/>
-            </geometry>
-        </collision>
-        <xacro:inertial_cylinder mass="${wheel_mass}" length="${wheel_thickness}" radius="${wheel_radius}">
-            <origin xyz="0 0 0" rpy="0 0 0"/>
-        </xacro:inertial_cylinder>
-    </link>
-    <gazebo reference="left_wheel_center">
-        <material>Gazebo/Black</material>
-    </gazebo>
-    <joint name="left_wheel_front_joint" type="continuous">
-        <parent link="base_link"/>
-        <child link="left_wheel_front"/>
-        <origin xyz="${wheel_spacing} ${wheel_offset_y} ${-wheel_offset_z}" rpy="-${pi/2} 0 0" />
-        <axis xyz="0 0 1"/>
-    </joint>
-    <link name="left_wheel_front">
-        <visual>
-            <geometry>
-                <cylinder radius="${wheel_radius}" length="${wheel_thickness}"/>
-            </geometry>
-            <material name="black"/>
-        </visual>
-        <collision>
-            <geometry>
-                <sphere radius="${wheel_radius}"/>
-            </geometry>
-        </collision>
-        <xacro:inertial_cylinder mass="${wheel_mass}" length="${wheel_thickness}" radius="${wheel_radius}">
-            <origin xyz="0 0 0" rpy="0 0 0"/>
-        </xacro:inertial_cylinder>
-    </link>
-    <gazebo reference="left_wheel_front">
-        <material>Gazebo/Black</material>
-    </gazebo>
-    <joint name="left_wheel_back_joint" type="continuous">
-        <parent link="base_link"/>
-        <child link="left_wheel_back"/>
-        <origin xyz="${-wheel_spacing} ${wheel_offset_y} ${-wheel_offset_z}" rpy="-${pi/2} 0 0" />
-        <axis xyz="0 0 1"/>
-    </joint>
-    <link name="left_wheel_back">
-        <visual>
-            <geometry>
-                <cylinder radius="${wheel_radius}" length="${wheel_thickness}"/>
-            </geometry>
-            <material name="black"/>
-        </visual>
-        <collision>
-            <geometry>
-                <sphere radius="${wheel_radius}"/>
-            </geometry>
-        </collision>
-        <xacro:inertial_cylinder mass="${wheel_mass}" length="${wheel_thickness}" radius="${wheel_radius}">
-            <origin xyz="0 0 0" rpy="0 0 0"/>
-        </xacro:inertial_cylinder>
-    </link>
-    <gazebo reference="left_wheel_back">
-        <material>Gazebo/Black</material>
-    </gazebo>
-    <!-- RIGHT WHEEL LINK -->
-    <joint name="right_wheel_center_joint" type="continuous">
-        <parent link="base_link"/>
-        <child link="right_wheel_center"/>
-        <origin xyz="0 ${-wheel_offset_y} ${-wheel_offset_z}" rpy="${pi/2} 0 0" />
-        <axis xyz="0 0 -1"/>
-    </joint>
-    <link name="right_wheel_center">
-        <visual>
-            <geometry>
-                <cylinder radius="${wheel_radius}" length="${wheel_thickness}"/>
-            </geometry>
-            <material name="black"/>
-        </visual>
-        <collision>
-            <geometry>
-                <sphere radius="${wheel_radius}"/>
-            </geometry>
-        </collision>
-        <xacro:inertial_cylinder mass="${wheel_mass}" length="${wheel_thickness}" radius="${wheel_radius}">
-            <origin xyz="0 0 0" rpy="0 0 0"/>
-        </xacro:inertial_cylinder>
-    </link>
-    <gazebo reference="right_wheel_center">
-        <material>Gazebo/Black</material>
-    </gazebo>
-    <joint name="right_wheel_front_joint" type="continuous">
-        <parent link="base_link"/>
-        <child link="right_wheel_front"/>
-        <origin xyz="${wheel_spacing} ${-wheel_offset_y} ${-wheel_offset_z}" rpy="${pi/2} 0 0" />
-        <axis xyz="0 0 -1"/>
-    </joint>
-    <link name="right_wheel_front">
-        <visual>
-            <geometry>
-                <cylinder radius="${wheel_radius}" length="${wheel_thickness}"/>
-            </geometry>
-            <material name="black"/>
-        </visual>
-        <collision>
-            <geometry>
-                <sphere radius="${wheel_radius}"/>
-            </geometry>
-        </collision>
-        <xacro:inertial_cylinder mass="${wheel_mass}" length="${wheel_thickness}" radius="${wheel_radius}">
-            <origin xyz="0 0 0" rpy="0 0 0"/>
-        </xacro:inertial_cylinder>
-    </link>
-    <gazebo reference="right_wheel_front">
-        <material>Gazebo/Black</material>
-    </gazebo>
-    <joint name="right_wheel_back_joint" type="continuous">
-        <parent link="base_link"/>
-        <child link="right_wheel_back"/>
-        <origin xyz="${-wheel_spacing} ${-wheel_offset_y} ${-wheel_offset_z}" rpy="${pi/2} 0 0" />
-        <axis xyz="0 0 -1"/>
-    </joint>
-    <link name="right_wheel_back">
-        <visual>
-            <geometry>
-                <cylinder radius="${wheel_radius}" length="${wheel_thickness}"/>
-            </geometry>
-            <material name="black"/>
-        </visual>
-        <collision>
-            <geometry>
-                <sphere radius="${wheel_radius}"/>
-            </geometry>
-        </collision>
-        <xacro:inertial_cylinder mass="${wheel_mass}" length="${wheel_thickness}" radius="${wheel_radius}">
-            <origin xyz="0 0 0" rpy="0 0 0"/>
-        </xacro:inertial_cylinder>
-    </link>
-    <gazebo reference="right_wheel_back">
-        <material>Gazebo/Black</material>
-    </gazebo>
     <link name="rack">
         <visual>
-            <origin xyz=" 0 0 0"/>
+            <origin xyz="0 0 0"/>
             <geometry>
-                <box size="0.6 0.37 0.47"/>
+                <box size="${rack_length} ${rack_width} ${rack_height}"/>
             </geometry>
             <material name="black_t"/>
@@ -236,15 +83,11 @@
             <origin xyz="0 0 0"/>
             <geometry>
-                <box size="${chassis_length*0.6} ${chassis_width*0.8} 0.5"/>
+                <box size="${rack_length} ${rack_width} ${rack_height}"/>
             </geometry>
         </collision>
-        <xacro:inertial_box mass="0.1" x="${chassis_length*0.6}" y="${chassis_width*0.8}" z="0.5">
+        <xacro:inertial_box mass="${rack_mass}"
+                            x="${rack_length}" y="${rack_width}" z="${rack_height}">
             <origin xyz="0 0 0" rpy="0 0 0"/>
         </xacro:inertial_box>
     </link>
-    <joint name="base2rack" type="fixed">
-        <parent link="base_link"/>
-        <child link="rack"/>
-        <origin xyz="0.02 0 0.25"/>
-    </joint>
 </robot>
