Commit message: implemented tracks using Gazebo's TrackedVehicle plugin

File: jo_description/urdf/track.xacro (robot description, xacro)
@@ -18,4 +18,5 @@
         <link name="back_${side}_roller">
             <visual>
+                <origin xyz="0 0 0" rpy="${-pi/2} ${-pi/2} 0"/>
                 <geometry>
                     <cylinder radius="${back_roller_radius}" length="${track_width}"/>
@@ -23,12 +24,13 @@
                 <material name="black"/>
             </visual>
-            <!-- <collision>
+            <collision>
+                <origin xyz="0 0 0" rpy="${-pi/2} ${-pi/2} 0"/>
                 <geometry>
                     <cylinder radius="${back_roller_radius}" length="${track_width}"/>
                 </geometry>
-                <material name="black"/>
-            </collision>      -->
+                <material name="orange"/>
+            </collision>
             <xacro:inertial_cylinder mass="0.01" radius="${back_roller_radius}" length="${track_width}">
-                    <origin xyz="0 0 0" rpy="0 0 0"/>
+                    <origin xyz="0 0 0" rpy="${-pi/2} ${-pi/2} 0"/>
             </xacro:inertial_cylinder>
         </link>
@@ -36,8 +38,9 @@
             <parent link="base_link"/>
             <child link="back_${side}_roller"/>
-            <origin xyz="${-chassis_length/2 - back_roller2chassis + back_roller_radius} ${(track_width/2 + chassis_width/2) * (1 if side == 'left' else -1)} ${-wheel_offset_z}" rpy="${pi/2} 0 0" />
+            <origin xyz="${-chassis_length/2 - back_roller2chassis + back_roller_radius} ${(track_width/2 + chassis_width/2) * (1 if side == 'left' else -1)} ${-chassis_height}" rpy="${pi/2} ${pi/2} ${pi/2}" />
         </joint>
         <link name="front_${side}_roller">
             <visual>
+                <origin xyz="0 0 0" rpy="${-pi/2} 0 0"/>
                 <geometry>
                     <cylinder radius="${front_roller_radius}" length="${track_width}"/>
@@ -45,12 +48,13 @@
                 <material name="black"/>
             </visual>
-            <!-- <collision>
+            <collision>
+                <origin xyz="0 0 0" rpy="${-pi/2} 0 0"/>
                 <geometry>
                     <cylinder radius="${front_roller_radius}" length="${track_width}"/>
                 </geometry>
-                <material name="black"/>
-            </collision>     -->
+                <material name="orange"/>
+            </collision>
             <xacro:inertial_cylinder mass="0.01" radius="${front_roller_radius}" length="${track_width}">
-                    <origin xyz="0 0 0" rpy="0 0 0"/>
+                    <origin xyz="0 0 0" rpy="${-pi/2} 0 0"/>
             </xacro:inertial_cylinder>
         </link>
@@ -58,8 +62,9 @@
             <parent link="back_${side}_roller"/>
             <child link="front_${side}_roller"/>
-            <origin xyz="${back2front_length} 0.0 0.0" rpy="0 0 ${pi/4}" />
+            <origin xyz="0.0 0.0 ${back2front_length}" rpy="0 0 0" />
         </joint>
         <link name="front_${side}_upper_roller">
             <visual>
+                <origin xyz="0 0 0" rpy="${-pi/2} ${-pi/4 - pi/3 - 17.7*pi/180} 0"/>
                 <geometry>
                     <cylinder radius="${front_upper_roller_radius}" length="${track_width}"/>
@@ -68,8 +73,9 @@
             </visual>
             <collision>
+                <origin xyz="0 0 0" rpy="${-pi/2} ${-pi/4 - pi/3 - 17.7*pi/180} 0"/>
                 <geometry>
                     <cylinder radius="${front_upper_roller_radius}" length="${track_width}"/>
                 </geometry>
-                <material name="black"/>
+                <material name="orange"/>
             </collision>
         </link>
@@ -77,5 +83,5 @@
             <parent link="front_${side}_roller"/>
             <child link="front_${side}_upper_roller"/>
-            <origin xyz="${front2upper_roller_length} 0.0 0.0" rpy="0 0 ${pi/4 + pi/3 + 17.7*pi/180}" />
+            <origin xyz="${-front2upper_roller_length * 0.7} 0.0 ${front2upper_roller_length * 0.7}" rpy="0 ${pi/4 + pi/3 + 17.7*pi/180} 0" />
         </joint>
         <link name="${side}_bottom_belt">
@@ -90,5 +96,5 @@
                     <box size="${belt_thickness} ${track_width} ${back2front_length}"/>
                 </geometry>
-                <material name="black"/>
+                <material name="orange"/>
             </collision>
             <xacro:inertial_box mass="0.01" x="${belt_thickness}" y="${track_width}" z="${back2front_length}">
@@ -99,27 +105,33 @@
             <parent link="back_${side}_roller"/>
             <child link="${side}_bottom_belt"/>
-            <origin xyz="${back2front_length/2} -0.065 0.0" rpy="${-pi/2} 0 ${-pi/2}" />
+            <origin xyz="0.065 0 ${back2front_length/2}" rpy="0 0 0" />
         </joint>
         <link name="${side}_front_bottom_belt">
             <visual>
-                <geometry>
-                    <box size="${front2upper_roller_length} ${belt_thickness} ${track_width}"/>
-                </geometry>
-                <material name="black"/>
-            </visual>
-            <collision>
-                <geometry>
-                    <box size="${front2upper_roller_length} ${belt_thickness} ${track_width}"/>
-                </geometry>
-                <material name="black"/>
-            </collision>
+                <origin xyz="0 0 0" rpy="0 ${-pi/4} 0"/>
+                <geometry>
+                    <box size="${belt_thickness} ${track_width} ${front2upper_roller_length}"/>
+                </geometry>
+                <material name="black"/>
+            </visual>
+            <collision>
+                <origin xyz="0 0 0" rpy="0 ${-pi/4} 0"/>
+                <geometry>
+                    <box size="${belt_thickness} ${track_width} ${front2upper_roller_length}"/>
+                </geometry>
+                <material name="orange"/>
+            </collision>
+            <xacro:inertial_box mass="0.01" x="${belt_thickness}" y="${track_width}" z="${front2upper_roller_length}">
+                    <origin xyz="0 0 0" rpy="0 ${-pi/4} 0"/>
+            </xacro:inertial_box>
         </link>
         <joint name="back_${side}_roller2${side}_front_bottom_belt" type="fixed">
             <parent link="front_${side}_roller"/>
             <child link="${side}_front_bottom_belt"/>
-            <origin xyz="${front2upper_roller_length/2} -0.065 0.0" rpy="0 0 0" />
+            <origin xyz="0.0 0.0 ${front2upper_roller_length/2}" rpy="0 0 0" />
         </joint>
         <link name="${side}_top_roller">
             <visual>
+                <origin xyz="0 0 0" rpy="${-pi/2} ${pi/6 + 2*pi/180} 0"/>
                 <geometry>
                     <cylinder radius="${upper_roller_radius}" length="${track_width}"/>
@@ -128,8 +140,9 @@
             </visual>
             <collision>
+                <origin xyz="0 0 0" rpy="${-pi/2} ${pi/6 + 2*pi/180} 0"/>
                 <geometry>
                     <cylinder radius="${upper_roller_radius}" length="${track_width}"/>
                 </geometry>
-                <material name="black"/>
+                <material name="orange"/>
             </collision>
         </link>
@@ -137,18 +150,18 @@
             <parent link="back_${side}_roller"/>
             <child link="${side}_top_roller"/>
-            <origin xyz="${back2top_roller_x} ${back2top_roller_y} 0" rpy="0 0 ${pi/6 + pi + 2*pi/180}" />
+            <origin xyz="${-back2top_roller_y} 0 ${back2top_roller_x}" rpy="0 ${-pi/6 - 2*pi/180} 0" />
         </joint>
         <link name="${side}_back_top_belt">
             <visual>
                 <geometry>
-                    <box size="${back2top_length} ${belt_thickness} ${track_width}"/>
-                </geometry>
-                <material name="black"/>
-            </visual>
-            <collision>
-                <geometry>
-                    <box size="${back2top_length} ${belt_thickness} ${track_width}"/>
-                </geometry>
-                <material name="black"/>
+                    <box size="${belt_thickness} ${track_width} ${back2top_length}"/>
+                </geometry>
+                <material name="black"/>
+            </visual>
+            <collision>
+                <geometry>
+                    <box size="${belt_thickness} ${track_width} ${back2top_length}"/>
+                </geometry>
+                <material name="orange"/>
             </collision>
         </link>
@@ -156,18 +169,18 @@
             <parent link="${side}_top_roller"/>
             <child link="${side}_back_top_belt"/>
-            <origin xyz="${back2top_length/2} -0.02 0.0" rpy="0 0 0" />
+            <origin xyz="-0.02 0.0 ${-back2top_length/2}" rpy="0 0 0" />
         </joint>
         <link name="${side}_front_top_belt">
             <visual>
                 <geometry>
-                    <box size="${top2front_upper_length} ${belt_thickness} ${track_width}"/>
-                </geometry>
-                <material name="black"/>
-            </visual>
-            <collision>
-                <geometry>
-                    <box size="${top2front_upper_length} ${belt_thickness} ${track_width}"/>
-                </geometry>
-                <material name="black"/>
+                    <box size="${top2front_upper_length} ${track_width} ${belt_thickness}"/>
+                </geometry>
+                <material name="black"/>
+            </visual>
+            <collision>
+                <geometry>
+                    <box size="${top2front_upper_length} ${track_width} ${belt_thickness}"/>
+                </geometry>
+                <material name="orange"/>
             </collision>
         </link>
@@ -175,7 +188,7 @@
             <parent link="front_${side}_upper_roller"/>
             <child link="${side}_front_top_belt"/>
-            <origin xyz="${top2front_upper_length/2} -0.065 0.0" rpy="0 0 0" />
-        </joint>
-        <!-- <gazebo reference="base2back_${side}_roller">
+            <origin xyz="${top2front_upper_length/2} 0.0 ${belt_thickness/2 + 0.005}" rpy="0 ${-pi/9} 0" />
+        </joint>
+        <gazebo reference="base2back_${side}_roller">
             <preserveFixedJoint>true</preserveFixedJoint>
         </gazebo>
@@ -186,12 +199,9 @@
                 <debug>0</debug>
             </plugin>
-        </gazebo> -->
-        <!-- <gazebo reference="back_${side}_roller">
-            <self_collide>false</self_collide>
-            <mu1>0.7</mu1>
-            <mu2>150</mu2>
-            <fdir1>0 1 0</fdir1>
-        </gazebo> -->
-        <!-- <gazebo reference="back_${side}_roller2front_${side}_roller">
+        </gazebo>
+        <gazebo reference="back_${side}_roller">
+            <self_collide>false</self_collide>
+        </gazebo>
+        <gazebo reference="back_${side}_roller2front_${side}_roller">
             <preserveFixedJoint>true</preserveFixedJoint>
         </gazebo>
@@ -202,5 +212,8 @@
                 <debug>0</debug>
             </plugin>
-        </gazebo> -->
+        </gazebo>
+        <gazebo reference="front_${side}_roller">
+            <self_collide>false</self_collide>
+        </gazebo>
         <gazebo reference="back_${side}_roller2${side}_bottom_belt">
             <preserveFixedJoint>true</preserveFixedJoint>
@@ -212,4 +225,20 @@
                 <debug>0</debug>
             </plugin>
+        </gazebo>
+        <gazebo reference="${side}_bottom_belt">
+            <self_collide>false</self_collide>
+        </gazebo>
+        <gazebo reference="back_${side}_roller2${side}_front_bottom_belt">
+            <preserveFixedJoint>true</preserveFixedJoint>
+        </gazebo>
+        <gazebo>
+            <plugin filename="gz-sim-track-controller-system"
+                    name="gz::sim::systems::TrackController">
+                <link>${side}_front_bottom_belt</link>
+                <debug>0</debug>
+            </plugin>
+        </gazebo>
+        <gazebo reference="${side}_front_bottom_belt">
+            <self_collide>false</self_collide>
         </gazebo>
         <!-- <gazebo reference="${side}_bottom_belt">

File: jo_description/urdf/velodyne.xacro (robot description, xacro)
@@ -4,5 +4,5 @@
     <xacro:property name="b2l_x" value="0.03" />
     <xacro:property name="b2l_y" value="0.0286" />
-    <xacro:property name="b2l_z" value="0.630" />
+    <xacro:property name="b2l_z" value="0.564" />
     <xacro:property name="b2l_R" value="0.0" />
     <xacro:property name="b2l_P" value="0.0" />
@@ -16,5 +16,5 @@
             <parent link="base_link"/>
             <child link="velodyne"/>
-            <origin xyz="${b2l_x} ${b2l_y} ${b2l_z}" rpy="${b2l_R} ${b2l_P} ${b2l_Y}"/>
+            <origin xyz="${b2l_x} ${b2l_y} ${b2l_z + lidar_len_h/2}" rpy="${b2l_R} ${b2l_P} ${b2l_Y}"/>
         </joint>
         <link name="velodyne">
@@ -30,5 +30,5 @@
                     <cylinder radius="${lidar_len_rad}" length="${lidar_len_h}"/>
                 </geometry>
-                <material name="orange"/>
+                <material name="blue"/>
             </visual>
             <xacro:inertial_cylinder mass="${lidar_mass}" radius="${lidar_len_rad}" length="${lidar_len_h}">
@@ -46,5 +46,5 @@
                     <update_on_paused_sim>false</update_on_paused_sim>
                     <topic>${namespace}/velodyne_points</topic>
-                    <frame>${namespace}/velodyne</frame>
+                    <frame>velodyne</frame>
                     <pattern_preset>Puck</pattern_preset>
                 </plugin>
