Commit message: removed wrong collisions

File: jo_description/urdf/track.xacro (robot description, xacro)
@@ -217,5 +217,5 @@
                     <cylinder radius="0.06" length="0.02"/>
                 </geometry>
-                <material name="red"/>
+                <material name="white"/>
             </visual>
             <visual name="box_2">
@@ -261,10 +261,4 @@
                 <material name="white"/>
             </visual>
-            <collision>
-                <geometry>
-                    <box size="${top2front_upper_length} ${track_width} 0.02"/>
-                </geometry>
-                <material name="orange"/>
-            </collision>
         </link>
         <joint name="back_${side}_roller2${side}_cover" type="fixed">
